Commit message: lidar updated

File: description/robot.urdf.xacro (robot description, xacro)
@@ -3,3 +3,4 @@
     <xacro:include filename="robot_core.xacro" />
     <xacro:include filename="gazebo_control.xacro" />
+    <xacro:include filename="lidar.xacro" />
 </robot>

File: description/robot_core.xacro (robot description, xacro)
@@ -154,24 +154,52 @@
 </gazebo>
 <!--/////////////////////////// lidar link //////////////////////// -->
-<joint name="lidar_joint" type="fixed">
-        <parent link="body_link"/>
-        <child link="lidar_link"/>
-        <origin xyz="0.1 0 0.32" rpy="0 0 0"/>
+    <joint name="laser_joint" type="fixed">
+            <parent link="body_link"/>
+            <child link="laser_frame"/>
+            <origin xyz="0.1 0 0.32" rpy="0 0 0"/>
     </joint>
-    <link name="lidar_link">
-        <visual>
-            <geometry>
-                <cylinder radius="0.05" length="0.04"/>
-            </geometry>
-            <material name="red"/>
-        </visual>
-        <collision>
-            <geometry>
-                <cylinder radius="0.05" length="0.04"/>
-            </geometry>
-        </collision>
-    </link>
-    <gazebo reference="lidar_link">
-    <material>Gazebo/Red</material>
-</gazebo>
+        <link name="laser_frame">
+            <visual>
+                <geometry>
+                    <cylinder radius="0.05" length="0.04"/>
+                </geometry>
+                <material name="red"/>
+            </visual>
+            <collision>
+                <geometry>
+                    <cylinder radius="0.05" length="0.04"/>
+                </geometry>
+            </collision>
+        </link>
+        <gazebo reference="laser_frame">
+        <material>Gazebo/Red</material>
+        </gazebo>
+   <gazebo reference="laser_frame">
+        <material>Gazebo/Red</material>
+        <sensor name="laser" type="ray">
+            <pose> 0 0 0 0 0 0 </pose>
+            <visualize>true</visualize>
+            <update_rate>10</update_rate>
+            <ray>
+                <scan>
+                    <horizontal>
+                        <samples>360</samples>
+                        <min_angle>-3.14</min_angle>
+                        <max_angle>3.14</max_angle>
+                    </horizontal>
+                </scan>
+                <range>
+                    <min>0.3</min>
+                    <max>12</max>
+                </range>
+            </ray>
+            <plugin name="laser_controller" filename="libgazebo_ros_ray_sensor.so">
+                <ros>
+                    <argument>~/out:=scan</argument>
+                </ros>
+                <output_type>sensor_msgs/LaserScan</output_type>
+                <frame_name>laser_frame</frame_name>
+            </plugin>
+        </sensor>
+    </gazebo>
 </robot>
