Commit message: upto ros2-control

File: description/lidar.xacro (robot description, xacro)
@@ -1,31 +1,37 @@
 <?xml version="1.0"?>
 <robot xmlns:xacro="http://www.ros.org/wiki/xacro" >
-<!--/////////////////////////// lidar link //////////////////////// -->
     <joint name="laser_joint" type="fixed">
-            <parent link="body_link"/>
-            <child link="laser_frame"/>
-            <origin xyz="0.1 0 0.32" rpy="0 0 0"/>
+        <parent link="body"/>
+        <child link="laser_frame"/>
+        <origin xyz="0.22 0.0 0.33" rpy="0 0 0"/>
     </joint>
-        <link name="laser_frame">
-            <visual>
-                <geometry>
-                    <cylinder radius="0.05" length="0.04"/>
-                </geometry>
-                <material name="red"/>
-            </visual>
-            <collision>
-                <geometry>
-                    <cylinder radius="0.05" length="0.04"/>
-                </geometry>
-            </collision>
-        </link>
-        <gazebo reference="laser_frame">
-        <material>Gazebo/Red</material>
-        </gazebo>
-   <gazebo reference="laser_frame">
+    <link name="laser_frame">
+        <visual>
+            <geometry>
+                <cylinder radius="0.05" length="0.04"/>
+            </geometry>
+            <material name="black"/>
+        </visual>
+        <visual>
+            <origin xyz="0 0 -0.05"/>
+            <geometry>
+                <cylinder radius="0.01" length="0.1"/>
+            </geometry>
+            <material name="red"/>
+        </visual>
+        <collision>
+            <geometry>
+                <cylinder radius="0.05" length="0.04"/>
+            </geometry>
+        </collision>
+        <xacro:inertial_cylinder mass="0.1" length="0.04" radius="0.05">
+            <origin xyz="0 0 0" rpy="0 0 0"/>
+        </xacro:inertial_cylinder>
+    </link>
+    <gazebo reference="laser_frame">
         <material>Gazebo/Red</material>
         <sensor name="laser" type="ray">
             <pose> 0 0 0 0 0 0 </pose>
-            <visualize>true</visualize>
+            <visualize>false</visualize>
             <update_rate>10</update_rate>
             <ray>

File: description/robot.urdf.xacro (robot description, xacro)
@@ -1,6 +1,14 @@
 <?xml version="1.0"?>
 <robot xmlns:xacro="http://www.ros.org/wiki/xacro"  name="agni_2">
-    <xacro:include filename="robot_core.xacro" />
-    <xacro:include filename="gazebo_control.xacro" />
+ <xacro:arg name="use_ros2_control" default="true"/>
+  <xacro:include filename="robot_core.xacro" />
+    <xacro:if value="$(arg use_ros2_control)">
+        <xacro:include filename="/home/base/dev_ws/src/agni_2/description/ros2_control.xacro" />
+    </xacro:if>
+    <xacro:unless value="$(arg use_ros2_control)">
+        <xacro:include filename="gazebo_control.xacro" />
+    </xacro:unless>
     <xacro:include filename="lidar.xacro" />
+    <xacro:include filename="camera.xacro" />
+    <!-- <xacro:include filename="depth_camera.xacro" /> -->
 </robot>

File: description/robot_core.xacro (robot description, xacro)
@@ -1,5 +1,20 @@
 <?xml version="1.0"?>
 <robot xmlns:xacro="http://www.ros.org/wiki/xacro" >
-<xacro:include filename="inertial_macros.xacro"/>
+     <xacro:include filename="/home/base/dev_ws/src/agni_2/description/inertial_macros.xacro"/>
+    <xacro:property name="body_length" value="0.3"/>
+    <xacro:property name="body_width" value="0.3"/>
+    <xacro:property name="body_height" value="0.3"/>
+    <xacro:property name="body_mass" value="1.5"/>
+    <xacro:property name="wheel_radius" value="0.0415"/>
+    <xacro:property name="wheel_thickness" value="0.035"/>
+    <xacro:property name="wheel_mass" value="0.05"/>
+    <xacro:property name="wheel_offset_x" value="0.15"/>
+    <xacro:property name="wheel_offset_y" value="0.15"/>
+    <xacro:property name="wheel_offset_z" value="0.01"/>
+    <xacro:property name="caster_wheel_radius" value="0.02"/>
+    <xacro:property name="caster_wheel_mass" value="0.01"/>
+    <xacro:property name="caster_wheel_offset_x" value="0.02"/>
+    <xacro:property name="r_caster_wheel_offset_x" value="0.28"/>
+    <xacro:property name="caster_wheel_offset_z" value="${wheel_offset_z - wheel_radius + caster_wheel_radius}"/>
   <material name="white">
       <color rgba="1 1 1 1"/>
@@ -19,187 +34,148 @@
 <!--/////////////////////////// base link //////////////////////// -->
   <link name="base_link">
+     <pose>0 0 0 0 0 -3.14159</pose>
+  </link>
+<!--/////////////////////////// base footprint link //////////////////////// -->
+ <joint name="base_footprint_joint" type="fixed">
+    <parent link="base_link"/>
+    <child link="base_footprint"/>
+    <origin xyz="0.0 0.0 0.0" rpy="0.0 0.0 0.0"/>
+  </joint>
+  <link name="base_footprint">
   </link>
 <!--/////////////////////////// body link //////////////////////// -->
-  <joint name="body_joint" type="fixed">
-    <parent link="base_link"/>
-    <child link="body_link"/>
-    <origin xyz="-0.15 0.0 0.0" rpy="0.0 0.0 0.0"/>
-  </joint>
-  <link name="body_link">
-    <visual>
-    <origin xyz="0.15 0.0 0.15" rpy="0.0 0.0 0.0"/>
-      <geometry>
-        <box size="0.3 0.3 0.3"/>
-      </geometry>
-      <material name="white"/>
-    </visual>
-    <collision>
-    <origin xyz="0.15 0.0 0.15" rpy="0.0 0.0 0.0"/>
-      <geometry>
-        <box size="0.3 0.3 0.3"/>
-      </geometry>
-    </collision>
-    <xacro:inertial_box mass="1.5" x="0.3" y="0.3" z="0.3">
-       <origin xyz="0.15 0.0 0.15" rpy="0.0 0.0 0.0"/>
-    </xacro:inertial_box>
-  </link>
- <gazebo reference="body_link">
-    <material>Gazebo/White</material>
-</gazebo>
+      <joint name="body_joint" type="fixed">
+        <parent link="base_link"/>
+        <child link="body"/>
+        <origin xyz="${-wheel_offset_x} 0 ${-wheel_offset_z}" />
+    </joint>
+    <link name="body">
+        <visual>
+            <origin xyz="${body_length/2} 0 ${body_height/2}"/>
+            <pose xyz="${body_length/2} 0 ${body_height/2}" rz="180.0"/>
+            <geometry>
+                <box size="${body_length} ${body_width} ${body_height}"/>
+            </geometry>
+            <material name="orange"/>
+        </visual>
+        <collision>
+            <origin xyz="${body_length/2} 0 ${body_height/2}"/>
+            <pose xyz="${body_length/2} 0 ${body_height/2}" rz="180.0"/>
+            <geometry>
+                <box size="${body_length} ${body_width} ${body_height}"/>
+            </geometry>
+        </collision>
+        <xacro:inertial_box mass="0.5" x="${body_length}" y="${body_width}" z="${body_height}">
+            <origin xyz="${body_length/2} 0 ${body_height/2}" rpy="0 0 0"/>
+        </xacro:inertial_box>
+    </link>
+    <gazebo reference="body">
+        <material>Gazebo/Orange</material>
+    </gazebo>
 <!--/////////////////////////// left wheel link //////////////////////// -->
- <joint name="left_wheel_joint" type="continuous">
- <parent link="body_link"/>
- <child link="left_wheel"/>
- <origin xyz="0.15 0.15 0.0" rpy="-1.57 0.0 0.0"/>
- <axis xyz="0.0 0.0 -1"/>
- </joint>
- <link name="left_wheel">
-  <visual>
-    <geometry>
-      <cylinder radius="0.0415" length="0.033"/>
-    </geometry>
-    <material name="blue"/>
-  </visual>
-  <collision>
-    <geometry>
-      <cylinder radius="0.0415" length="0.033"/>
-    </geometry>
-  </collision>
-  <xacro:inertial_cylinder mass="0.1" length="0.033" radius="0.0415">
-        <origin xyz="0 0 0" rpy="0 0 0"/>
-  </xacro:inertial_cylinder>
- </link>
- <gazebo reference="left_wheel">
-    <material>Gazebo/Blue</material>
-</gazebo>
+<joint name="left_wheel_joint" type="continuous">
+        <parent link="base_link"/>
+        <child link="left_wheel"/>
+        <origin xyz="0 ${wheel_offset_y} 0" rpy="${-pi/2} 0 0" />
+        <axis xyz="0 0 1"/>
+    </joint>
+    <link name="left_wheel">
+        <visual>
+            <geometry>
+                <cylinder radius="${wheel_radius}" length="${wheel_thickness}"/>
+            </geometry>
+            <material name="blue"/>
+        </visual>
+        <collision>
+            <geometry>
+                <sphere radius="${wheel_radius}"/>
+            </geometry>
+        </collision>
+        <xacro:inertial_cylinder mass="${wheel_mass}" length="${wheel_thickness}" radius="${wheel_radius}">
+            <origin xyz="0 0 0" rpy="0 0 0"/>
+        </xacro:inertial_cylinder>
+    </link>
+    <gazebo reference="left_wheel">
+        <material>Gazebo/Blue</material>
+    </gazebo>
  <!--/////////////////////////// right wheel link //////////////////////// -->
- <joint name="right_wheel_joint" type="continuous">
- <parent link="body_link"/>
- <child link="right_wheel"/>
- <origin xyz="0.15 -0.15 0.0" rpy="1.57 0.0 0.0"/>
- <axis xyz="0.0 0.0 1"/>
- </joint>
- <link name="right_wheel">
-  <visual>
-    <geometry>
-      <cylinder radius="0.0415" length="0.033"/>
-    </geometry>
-    <material name="blue"/>
-  </visual>
-   <collision>
-    <geometry>
-      <cylinder radius="0.0415" length="0.033"/>
-    </geometry>
-  </collision>
-  <xacro:inertial_cylinder mass="0.1" length="0.033" radius="0.0415">
-        <origin xyz="0 0 0" rpy="0 0 0"/>
-  </xacro:inertial_cylinder>
- </link>
- <gazebo reference="right_wheel">
-    <material>Gazebo/Blue</material>
-</gazebo>
+  <joint name="right_wheel_joint" type="continuous">
+        <parent link="base_link"/>
+        <child link="right_wheel"/>
+        <origin xyz="0 ${-wheel_offset_y} 0" rpy="${pi/2} 0 0" />
+        <axis xyz="0 0 -1"/>
+    </joint>
+    <link name="right_wheel">
+        <visual>
+            <geometry>
+                <cylinder radius="${wheel_radius}" length="${wheel_thickness}"/>
+            </geometry>
+            <material name="blue"/>
+        </visual>
+        <collision>
+            <geometry>
+                <sphere radius="${wheel_radius}"/>
+            </geometry>
+        </collision>
+        <xacro:inertial_cylinder mass="${wheel_mass}" length="${wheel_thickness}" radius="${wheel_radius}">
+            <origin xyz="0 0 0" rpy="0 0 0"/>
+        </xacro:inertial_cylinder>
+    </link>
+    <gazebo reference="right_wheel">
+        <material>Gazebo/Blue</material>
+    </gazebo>
   <!--/////////////////////////// f_caster wheel link //////////////////////// -->
  <joint name="f_caster_wheel_joint" type="fixed">
- <parent link="body_link"/>
- <child link="f_caster_wheel"/>
- <origin xyz="0.24 0.0 0.0" rpy="0.0 0.0 0.0"/>
- </joint>
- <link name="f_caster_wheel">
-  <visual>
-    <geometry>
-      <sphere radius="0.04"/>
-    </geometry>
-    <material name="black"/>
-  </visual>
-  <collision>
-    <geometry>
-      <sphere radius="0.04"/>
-    </geometry>
-  </collision>
-  <xacro:inertial_sphere mass="0.1" radius="0.04">
+        <parent link="body"/>
+        <child link="f_caster_wheel"/>
+        <origin xyz="${caster_wheel_offset_x} 0 ${caster_wheel_offset_z}"/>
+    </joint>
+    <link name="f_caster_wheel">
+        <visual>
+            <geometry>
+                <sphere radius="${caster_wheel_radius}"/>
+            </geometry>
+            <material name="white"/>
+        </visual>
+        <collision>
+            <geometry>
+                <sphere radius="${caster_wheel_radius}"/>
+            </geometry>
+        </collision>
+        <xacro:inertial_sphere mass="${caster_wheel_mass}" radius="${caster_wheel_radius}">
             <origin xyz="0 0 0" rpy="0 0 0"/>
         </xacro:inertial_sphere>
- </link>
-  <gazebo reference="f_caster_wheel">
-    <material>Gazebo/Black</material>
-    <mu1 value="0.001"/>
-    <mu2 value="0.001"/>
-</gazebo>
+    </link>
+    <gazebo reference="f_caster_wheel">
+        <material>Gazebo/White</material>
+        <mu1 value="0.001"/>
+        <mu2 value="0.001"/>
+    </gazebo>
    <!--/////////////////////////// r_caster wheel link //////////////////////// -->
  <joint name="r_caster_wheel_joint" type="fixed">
- <parent link="body_link"/>
- <child link="r_caster_wheel"/>
- <origin xyz="0.06 0.0 0.0" rpy="0.0 0.0 0.0"/>
- </joint>
- <link name="r_caster_wheel">
-  <visual>
-    <geometry>
-      <sphere radius="0.04"/>
-    </geometry>
-    <material name="black"/>
-  </visual>
-  <collision>
-    <geometry>
-      <sphere radius="0.04"/>
-    </geometry>
-  </collision>
-<xacro:inertial_sphere mass="0.1" radius="0.04">
-        <origin xyz="0 0 0" rpy="0 0 0"/>
-</xacro:inertial_sphere>
- </link>
-   <gazebo reference="r_caster_wheel">
-    <material>Gazebo/Black</material>
-    <mu1 value="0.001"/>
-    <mu2 value="0.001"/>
-</gazebo>
-<!--/////////////////////////// lidar link //////////////////////// -->
-    <joint name="laser_joint" type="fixed">
-            <parent link="body_link"/>
-            <child link="laser_frame"/>
-            <origin xyz="0.1 0 0.32" rpy="0 0 0"/>
+        <parent link="body"/>
+        <child link="r_caster_wheel"/>
+        <origin xyz="${r_caster_wheel_offset_x} 0 ${caster_wheel_offset_z}"/>
     </joint>
-        <link name="laser_frame">
-            <visual>
-                <geometry>
-                    <cylinder radius="0.05" length="0.04"/>
-                </geometry>
-                <material name="red"/>
-            </visual>
-            <collision>
-                <geometry>
-                    <cylinder radius="0.05" length="0.04"/>
-                </geometry>
-            </collision>
-        </link>
-        <gazebo reference="laser_frame">
-        <material>Gazebo/Red</material>
-        </gazebo>
-   <gazebo reference="laser_frame">
-        <material>Gazebo/Red</material>
-        <sensor name="laser" type="ray">
-            <pose> 0 0 0 0 0 0 </pose>
-            <visualize>true</visualize>
-            <update_rate>10</update_rate>
-            <ray>
-                <scan>
-                    <horizontal>
-                        <samples>360</samples>
-                        <min_angle>-3.14</min_angle>
-                        <max_angle>3.14</max_angle>
-                    </horizontal>
-                </scan>
-                <range>
-                    <min>0.3</min>
-                    <max>12</max>
-                </range>
-            </ray>
-            <plugin name="laser_controller" filename="libgazebo_ros_ray_sensor.so">
-                <ros>
-                    <argument>~/out:=scan</argument>
-                </ros>
-                <output_type>sensor_msgs/LaserScan</output_type>
-                <frame_name>laser_frame</frame_name>
-            </plugin>
-        </sensor>
+    <link name="r_caster_wheel">
+        <visual>
+            <geometry>
+                <sphere radius="${caster_wheel_radius}"/>
+            </geometry>
+            <material name="white"/>
+        </visual>
+        <collision>
+            <geometry>
+                <sphere radius="${caster_wheel_radius}"/>
+            </geometry>
+        </collision>
+        <xacro:inertial_sphere mass="${caster_wheel_mass}" radius="${caster_wheel_radius}">
+            <origin xyz="0 0 0" rpy="0 0 0"/>
+        </xacro:inertial_sphere>
+    </link>
+    <gazebo reference="r_caster_wheel">
+        <material>Gazebo/White</material>
+        <mu1 value="0.001"/>
+        <mu2 value="0.001"/>
     </gazebo>
 </robot>
