Commit message: final

File: description/camera.xacro (robot description, xacro)
@@ -1,4 +1,4 @@
 <?xml version="1.0"?>
-<robot xmlns:xacro="http://www.ros.org/wiki/xacro" >
+<robot xmlns:xacro="http://www.ros.org/wiki/xacro">
     <joint name="camera_joint" type="fixed">
         <parent link="body"/>

File: description/gazebo_control.xacro (robot description, xacro)
@@ -6,5 +6,5 @@
             <left_joint>left_wheel_joint</left_joint>
             <right_joint>right_wheel_joint</right_joint>
-            <wheel_separation>0.3</wheel_separation>
+            <wheel_separation>0.345</wheel_separation>
             <wheel_diameter>0.083</wheel_diameter>
             <!-- Limits -->

File: description/lidar.xacro (robot description, xacro)
@@ -11,5 +11,5 @@
                 <cylinder radius="0.05" length="0.04"/>
             </geometry>
-            <material name="black"/>
+            <material name="red"/>
         </visual>
         <visual>
@@ -33,5 +33,5 @@
         <sensor name="laser" type="ray">
             <pose> 0 0 0 0 0 0 </pose>
-            <visualize>false</visualize>
+            <visualize>true</visualize>
             <update_rate>10</update_rate>
             <ray>

File: description/robot.urdf.xacro (robot description, xacro)
@@ -2,13 +2,14 @@
 <robot xmlns:xacro="http://www.ros.org/wiki/xacro"  name="agni_2">
  <xacro:arg name="use_ros2_control" default="true"/>
-  <xacro:include filename="robot_core.xacro" />
+ <xacro:arg name="sim_mode" default="false"/>
+  <xacro:include filename="/home/robot/dev_ws/src/agni_2/description/robot_core.xacro" />
     <xacro:if value="$(arg use_ros2_control)">
-        <xacro:include filename="/home/base/dev_ws/src/agni_2/description/ros2_control.xacro" />
+        <xacro:include filename="/home/robot/dev_ws/src/agni_2/description/ros2_control.xacro" />
     </xacro:if>
     <xacro:unless value="$(arg use_ros2_control)">
-        <xacro:include filename="gazebo_control.xacro" />
+        <xacro:include filename="/home/robot/dev_ws/src/agni_2/description/gazebo_control.xacro" />
     </xacro:unless>
     <xacro:include filename="lidar.xacro" />
-    <xacro:include filename="camera.xacro" />
+    <!--<xacro:include filename="/home/robot/dev_ws/src/agni_2/description/camera.xacro" /> -->
     <!-- <xacro:include filename="depth_camera.xacro" /> -->
 </robot>

File: description/robot_core.xacro (robot description, xacro)
@@ -1,19 +1,18 @@
 <?xml version="1.0"?>
 <robot xmlns:xacro="http://www.ros.org/wiki/xacro" >
-     <xacro:include filename="/home/base/dev_ws/src/agni_2/description/inertial_macros.xacro"/>
+     <xacro:include filename="/home/robot/dev_ws/src/agni_2/description/inertial_macros.xacro"/>
     <xacro:property name="body_length" value="0.3"/>
     <xacro:property name="body_width" value="0.3"/>
     <xacro:property name="body_height" value="0.3"/>
-    <xacro:property name="body_mass" value="1.5"/>
+    <xacro:property name="body_mass" value="5"/>
     <xacro:property name="wheel_radius" value="0.0415"/>
     <xacro:property name="wheel_thickness" value="0.035"/>
     <xacro:property name="wheel_mass" value="0.05"/>
-    <xacro:property name="wheel_offset_x" value="0.15"/>
-    <xacro:property name="wheel_offset_y" value="0.15"/>
+    <xacro:property name="wheel_offset_x" value="0.226"/>
+    <xacro:property name="wheel_offset_y" value="0.1485"/>
     <xacro:property name="wheel_offset_z" value="0.01"/>
     <xacro:property name="caster_wheel_radius" value="0.02"/>
     <xacro:property name="caster_wheel_mass" value="0.01"/>
     <xacro:property name="caster_wheel_offset_x" value="0.02"/>
-    <xacro:property name="r_caster_wheel_offset_x" value="0.28"/>
     <xacro:property name="caster_wheel_offset_z" value="${wheel_offset_z - wheel_radius + caster_wheel_radius}"/>
   <material name="white">
@@ -48,5 +47,5 @@
         <parent link="base_link"/>
         <child link="body"/>
-        <origin xyz="${-wheel_offset_x} 0 ${-wheel_offset_z}" />
+        <origin xyz="${-wheel_offset_x} 0 ${-wheel_offset_z}" rpy="0 0 0"/>
     </joint>
     <link name="body">
@@ -71,5 +70,5 @@
     </link>
     <gazebo reference="body">
-        <material>Gazebo/Orange</material>
+        <material>Gazebo/Blue</material>
     </gazebo>
 <!--/////////////////////////// left wheel link //////////////////////// -->
@@ -97,5 +96,5 @@
     </link>
     <gazebo reference="left_wheel">
-        <material>Gazebo/Blue</material>
+        <material>Gazebo/Black</material>
     </gazebo>
  <!--/////////////////////////// right wheel link //////////////////////// -->
@@ -123,13 +122,13 @@
     </link>
     <gazebo reference="right_wheel">
-        <material>Gazebo/Blue</material>
+        <material>Gazebo/Black</material>
     </gazebo>
-  <!--/////////////////////////// f_caster wheel link //////////////////////// -->
- <joint name="f_caster_wheel_joint" type="fixed">
+  <!--/////////////////////////// caster wheel link //////////////////////// -->
+ <joint name="caster_wheel_joint" type="fixed">
         <parent link="body"/>
-        <child link="f_caster_wheel"/>
+        <child link="caster_wheel"/>
         <origin xyz="${caster_wheel_offset_x} 0 ${caster_wheel_offset_z}"/>
     </joint>
-    <link name="f_caster_wheel">
+    <link name="caster_wheel">
         <visual>
             <geometry>
@@ -147,32 +146,5 @@
         </xacro:inertial_sphere>
     </link>
-    <gazebo reference="f_caster_wheel">
-        <material>Gazebo/White</material>
-        <mu1 value="0.001"/>
-        <mu2 value="0.001"/>
-    </gazebo>
-   <!--/////////////////////////// r_caster wheel link //////////////////////// -->
- <joint name="r_caster_wheel_joint" type="fixed">
-        <parent link="body"/>
-        <child link="r_caster_wheel"/>
-        <origin xyz="${r_caster_wheel_offset_x} 0 ${caster_wheel_offset_z}"/>
-    </joint>
-    <link name="r_caster_wheel">
-        <visual>
-            <geometry>
-                <sphere radius="${caster_wheel_radius}"/>
-            </geometry>
-            <material name="white"/>
-        </visual>
-        <collision>
-            <geometry>
-                <sphere radius="${caster_wheel_radius}"/>
-            </geometry>
-        </collision>
-        <xacro:inertial_sphere mass="${caster_wheel_mass}" radius="${caster_wheel_radius}">
-            <origin xyz="0 0 0" rpy="0 0 0"/>
-        </xacro:inertial_sphere>
-    </link>
-    <gazebo reference="r_caster_wheel">
+    <gazebo reference="caster_wheel">
         <material>Gazebo/White</material>
         <mu1 value="0.001"/>

File: description/ros2_control.xacro (robot description, xacro)
@@ -1,4 +1,5 @@
 <?xml version="1.0"?>
 <robot xmlns:xacro="http://www.ros.org/wiki/xacro">
+    <xacro:unless value="$(arg sim_mode)">
         <ros2_control name="GazeboSystem" type="system">
             <hardware>
@@ -22,4 +23,28 @@
             </joint>
         </ros2_control>
+        </xacro:unless>
+         <xacro:if value="$(arg sim_mode)">
+        <ros2_control name="GazeboSystem" type="system">
+            <hardware>
+                <plugin>gazebo_ros2_control/GazeboSystem</plugin>
+            </hardware>
+            <joint name="left_wheel_joint">
+                <command_interface name="velocity">
+                    <param name="min">-10</param>
+                    <param name="max">10</param>
+                </command_interface>
+                <state_interface name="velocity"/>
+                <state_interface name="position"/>
+            </joint>
+            <joint name="right_wheel_joint">
+                <command_interface name="velocity">
+                    <param name="min">-10</param>
+                    <param name="max">10</param>
+                </command_interface>
+                <state_interface name="velocity"/>
+                <state_interface name="position"/>
+            </joint>
+        </ros2_control>
+    </xacro:if>
     <gazebo>
         <plugin name="gazebo_ros2_control" filename="libgazebo_ros2_control.so">
